Commit message: Update launch

File: pinky_description/urdf/camera.xacro (robot description, xacro)
@@ -6,8 +6,9 @@
             <camera name="camera">
                 <pose>0 0 0 0 -1.5707 0</pose>
+                <update_rate>60</update_rate>
                 <horizontal_fov>1.08</horizontal_fov>
                 <image>
-                    <width>1280</width>
-                    <height>720</height>
+                    <width>640</width>
+                    <height>360</height>
                     <format>R8G8B8</format>
                 </image>

File: pinky_description/urdf/robot_core.xacro (robot description, xacro)
@@ -24,5 +24,5 @@
         <inertial>
             <origin xyz="-0.02 0 0.028" rpy="0 0 0"/>
-            <mass value="0.5"/>
+            <mass value="2.0"/>
             <inertia ixx="0.01" ixy="0" ixz="0" iyy="0.01" iyz="0" izz="0.01"/>
         </inertial>
@@ -49,5 +49,5 @@
         <inertial>
             <origin xyz="0 0 0" rpy="0 0 0"/>
-            <mass value="0.3"/>
+            <mass value="0.2"/>
             <inertia ixx="0.1" ixy="0" ixz="0" iyy="0.1" iyz="0" izz="0.1"/>
         </inertial>
@@ -74,5 +74,5 @@
         <inertial>
             <origin xyz="0 0 0" rpy="0 0 0"/>
-            <mass value="0.3"/>
+            <mass value="0.2"/>
             <inertia ixx="0.1" ixy="0" ixz="0" iyy="0.1" iyz="0" izz="0.1"/>
         </inertial>
